File: esp8266-iotmaker.kicad_pcb (KiCad board)
At the start: 2 copper layers, 66 x 30.5 mm, 67 parts, among them J1 CONN_01X04, J2 CONN_01X02, J3 CONN_01X08, J4 CONN_01X06, J5 CONN_01X08, J6 CONN_01X04, Q1 S8050, Q2 S8050, SW1 SW_Push, SW2 SW_Push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

Commit message: add pcb
Parts:
- added D3: LED, LEDs:LED_0603, F.Cu at (160.0, 124.4)
- moved J4 20.3 mm to (161.5, 112.8)
- moved J5 15.2 mm to (141.2, 112.8)
- moved R7 5.26 mm to (157.4, 107.5), turned to 0 degrees
- moved C11 5.24 mm to (157.4, 109.1), turned to 0 degrees
- moved R14 4.60 mm to (152.2, 108.5), turned to 90 degrees
- moved R3 2.89 mm to (154.0, 108.5), turned to 270 degrees
- moved U4 1.84 mm to (176.6, 106.1), turned to 270 degrees
- moved C8 1.37 mm to (135.2, 93.5), turned to 90 degrees
- moved C9 1.27 mm to (138.9, 93.5), turned to 90 degrees
- moved C10 1.27 mm to (140.7, 93.5), turned to 90 degrees
- moved Q1 1.22 mm to (145.9, 106.1), turned to 270 degrees
- moved C6 1.13 mm to (137.0, 93.4), turned to 90 degrees
- moved D7 1.08 mm to (132.3, 87.9)
- moved D4 1.07 mm to (168.7, 106.4)
- moved R11 1.02 mm to (161.4, 108.9)
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Connections:
- J3 pad 1: GPIO14 -> GPIO13
- J3 pad 2: GPIO12 -> GPIO15
- J3 pad 3: GPIO13 -> GPIO12
- J3 pad 4: GPIO15 -> GPIO14
Routing:
- net GND: track 0.00 -> 172.1 mm, vias 0 -> 2
- net 3V3: track 0.00 -> 134.2 mm
- net GPIO16: track 0.00 -> 94.0 mm, vias 0 -> 1
- net 5V: track 0.00 -> 57.6 mm, vias 0 -> 2
- net GPIO0: track 0.00 -> 50.2 mm, vias 0 -> 2
- net GPIO4: track 0.00 -> 46.9 mm, vias 0 -> 1
- net Net-(C12-Pad1): track 0.00 -> 43.6 mm
- net GPIO2: track 0.00 -> 39.4 mm, vias 0 -> 1
- net GPIO10: track 0.00 -> 37.1 mm, vias 0 -> 2
- net SCLK: track 0.00 -> 29.8 mm, vias 0 -> 2
- net Net-(R3-Pad1): track 0.00 -> 29.6 mm, vias 0 -> 2
- net RTS: track 0.00 -> 29.4 mm
- net GPIO13: track 0.00 -> 27.5 mm, vias 0 -> 1
- net MOSI: track 0.00 -> 27.3 mm, vias 0 -> 2
- net Net-(BT1-Pad1): track 0.00 -> 25.7 mm
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Other:
- net class Default: trace_width 0.25 -> 0.254; via_dia 0.6 -> 1.1; via_drill 0.4 -> 0.6

Commit message: update footprint
Parts:
- removed D3: LED, LEDs:LED_0603
- removed R16: 470, esp8266:R_0603
- added C19: C, esp8266:C_0603, F.Cu at (160.9, 94.9)
- added C20: C, esp8266:C_0603, F.Cu at (162.8, 94.9)
- added C21: C, esp8266:C_0603, F.Cu at (144.7, 88.7)
- added C22: C, esp8266:C_0603, F.Cu at (144.7, 90.5)
- C12, C15: value 10uF -> C; footprint Capacitors_Tantalum_SMD:CP_Tantalum_Case-A_EIA-3216-18_Reflow -> esp8266:C_0603
- C14, C18: value 22uF -> C; footprint Capacitors_Tantalum_SMD:CP_Tantalum_Case-A_EIA-3216-18_Reflow -> esp8266:C_0603
- moved J6 36.6 mm to (173.7, 85.6)
- moved R15 32.9 mm to (139.7, 112.6)
- moved J3 30.9 mm to (143.3, 112.5)
- moved R6 27.4 mm to (152.5, 106.2), turned to 180 degrees
- moved J2 27.4 mm to (163.6, 112.5)
- moved J5 27.3 mm to (143.3, 85.6)
- moved R14 24.2 mm to (168.7, 90.7), turned to 180 degrees
- moved R3 22.6 mm to (175.6, 101.5), turned to 0 degrees
- moved R7 21.9 mm to (168.6, 88.6), turned to 180 degrees
- moved C11 20.7 mm to (164.7, 89.7)
- moved C15 20.0 mm to (144.7, 93.6), turned to 180 degrees
- moved D4 18.8 mm to (159.3, 90.1)
- moved C13 16.9 mm to (132.7, 88.5), turned to 180 degrees
- moved R11 16.3 mm to (168.5, 94.2), turned to 180 degrees
- moved C18 16.3 mm to (144.7, 95.4), turned to 180 degrees
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Connections:
- C12 pad 1: Net-(C12-Pad1) -> VBAT
- C14 pad 1: 5V -> VBAT
- C15 pad 1: VBAT -> Net-(C15-Pad1)
- C18 pad 1: 3V3 -> Net-(C15-Pad1)
- D4 pad 1: Net-(C12-Pad1) -> Net-(C15-Pad1)
- D5 pad 1: Net-(C12-Pad1) -> Net-(C15-Pad1)
- J1 pad 1: GPIO0 -> GPIO16
- J1 pad 2: GPIO2 -> ADC_EX
- J1 pad 3: 3V3 -> GND
- J1 pad 4: GND -> 3V3
- J2 pad 1: GPIO16 -> GPIO2
- J2 pad 2: ADC_EX -> GPIO0
- J3 pad 1: GPIO13 -> GPIO14
- J3 pad 2: GPIO15 -> GPIO12
- J3 pad 3: GPIO12 -> GPIO13
- J3 pad 4: GPIO14 -> GPIO15
- J4 pad 5: MISO -> SCLK
- J4 pad 6: SCLK -> MISO
- Q1 pad 3: EN -> REST
- U7 pad 3: Net-(C12-Pad1) -> Net-(C15-Pad1)
Routing:
- net GND: track 172.1 -> 325.7 mm, vias 2 -> 14
- net REST: track 10.6 -> 80.4 mm, vias 0 -> 1
- net VBAT: track 12.9 -> 74.8 mm, vias 0 -> 2
- net TXD: track 0.00 -> 61.7 mm, vias 0 -> 2
- net RXD: track 0.00 -> 51.7 mm, vias 0 -> 2
- net Net-(C12-Pad1): track 43.6 -> 0.00 mm
- net 3V3: track 134.2 -> 174.2 mm, vias 0 -> 8
- net EN: track 5.71 -> 42.1 mm, vias 0 -> 2
- net 5V: track 57.6 -> 29.5 mm, vias 2 -> 0
- net Net-(R3-Pad1): track 29.6 -> 2.82 mm, vias 2 -> 0
- net Net-(C15-Pad1): track 0.00 -> 24.3 mm
- net GPIO15: track 5.01 -> 28.9 mm, vias 0 -> 1
- net VUSB: track 15.4 -> 38.7 mm, vias 0 -> 2
- net GPIO5: track 0.00 -> 22.8 mm, vias 0 -> 1
- net RTS: track 29.4 -> 8.07 mm
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- added copper zone on B.Cu, net GND
- added copper zone on F.Cu, net GND
Other:
- board size 66 x 30.5 mm -> 66.3 x 30.7 mm
