File: esp8266-iotmaker.sch (KiCad schematic (older format))
At the start: 52 parts, among them Q1 S8050, Q2 S8050, SW1 SW_Push, SW2 SW_Push, U1 usb_mini_b, U2 chip-esp8266, U3 CP2102, U4 25Q32, U5 MCP6001, U6 AMS1117-3.3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

Commit message: xap xep linh kien'
Parts:
- removed AE1: Antenna, symbol Antenna
- removed D3: D_Schottky, symbol D_Schottky
- removed D4: LED, symbol LED
- removed D5: D_Schottky_ALT, symbol D_Schottky_ALT
- removed U5: MCP6001, symbol MCP6001
- removed U7: MOSFET-P, symbol MOSFET-P
- added AE1: Antenna_Shield, esp8266:anten, symbol Antenna_Shield
- added BT1: Battery, Pin_Headers:Pin_Header_Straight_2x01_Pitch2.00mm, symbol Battery_Cell
- added C15: 10uF, Capacitors_Tantalum_SMD:CP_Tantalum_Case-A_EIA-3216-18_Reflow, symbol CP1
- added C16: 4.7uF, esp8266:C_0603, symbol C
- added C17: 1uF, esp8266:C_0603, symbol C
- added C18: 22uF, Capacitors_Tantalum_SMD:CP_Tantalum_Case-A_EIA-3216-18_Reflow, symbol CP1
- added D3: LED, LEDs:LED_0603, symbol LED_Small_ALT
- added D4, D5: SS34, esp8266:do214aa-g, symbol D_Schottky_Small
- added D7: BAT60JFILM, Diodes_SMD:D_SOD-123, symbol D_Schottky_Small
- added D8: LED, LEDs:LED_0603, symbol LED_Small
- added J1, J6: CONN_01X04, Pin_Headers:Pin_Header_Straight_1x04_Pitch2.54mm, symbol CONN_01X04
- added J2: CONN_01X02, Pin_Headers:Pin_Header_Straight_1x02_Pitch2.54mm, symbol CONN_01X02
- added J3, J5: CONN_01X08, Pin_Headers:Pin_Header_Straight_1x08_Pitch2.54mm, symbol CONN_01X08
- added J4: CONN_01X06, Pin_Headers:Pin_Header_Straight_1x06_Pitch2.54mm, symbol CONN_01X06
- added R19: 100k, esp8266:R_0603, symbol R
- added R20: 2K, esp8266:R_0603, symbol R
- added U5: mcp73831, TO_SOT_Packages_SMD:SOT-23-5, symbol mcp73831
- added U7: AMS1117-3.3, TO_SOT_Packages_SMD:SOT-223, symbol AMS1117-3.3
- added U8: MOSFET-P, esp8266:SOT-23_standar, symbol MOSFET-P
- C1, C10, C11, C3, C4, C5, C6, C7, C8, C9: footprint (none) -> esp8266:C_0603
- C12, C14: footprint (none) -> Capacitors_Tantalum_SMD:CP_Tantalum_Case-A_EIA-3216-18_Reflow
- C13: value 100nF -> 4.7uF; footprint (none) -> esp8266:C_0603
- C2: value C -> 5.6pF; footprint (none) -> esp8266:C_0603
- D1: footprint (none) -> LEDs:LED_0603
- D2: footprint (none) -> Diodes_SMD:D_SOD-323_HandSoldering
- L1, L2: footprint (none) -> Inductors_SMD:L_0603
- Q1, Q2: footprint TO_SOT_Packages_THT:TO-92_Molded_Narrow -> esp8266:SOT-23_standar
- R1, R10, R11, R12, R13, R14, R15, R18, R2, R3, R4, R5, R6, R7, R8, R9: footprint (none) -> esp8266:R_0603
- R16: value 10k -> 470; footprint (none) -> esp8266:R_0603
- R17: value 10k -> 2K; footprint (none) -> esp8266:R_0603
- SW1, SW2: footprint (none) -> esp8266:Tact_Switch_TS6X3.6
- U1: footprint (none) -> USB_Micro-B
- U2: footprint (none) -> esp8266:esp8266ex
- U3: footprint (none) -> Housings_DFN_QFN:QFN-28-1EP_5x5mm_Pitch0.5mm
- U4: footprint (none) -> Housings_SOIC:SOIJ-8_5.3x5.3mm_Pitch1.27mm
- U6: footprint SOT-223 -> TO_SOT_Packages_SMD:SOT-223
- Y1: footprint (none) -> Crystals:Crystal_SMD_2016-4pin_2.0x1.6mm
Connections:
- net labels added: VIN
- wire segments 202 -> 258
Other:
- note added: "ESP8266EX"
- note added: "OLED"
- note added: "SPI FLASH"
- note removed: "ESP12F"
- moved on the sheet: C12, C14, D2, R12, R13, R8

Commit message: update footprint
Parts:
- removed C12, C15: 10uF, Capacitors_Tantalum_SMD:CP_Tantalum_Case-A_EIA-3216-18_Reflow, symbol CP1
- removed C14, C18: 22uF, Capacitors_Tantalum_SMD:CP_Tantalum_Case-A_EIA-3216-18_Reflow, symbol CP1
- added C12, C14, C15, C18, C19, C20, C21, C22: C, esp8266:C_0603, symbol C
- U1: footprint USB_Micro-B -> esp8266:USB_Micro-B
Connections:
- net 3V3: now also J1.4 (P4), C19.1, C20.1; no longer J1.3 (P3)
- net 5V: now also C21.1, C22.1
- net ADC_EX: now also J1.2 (P2); no longer J2.2 (P2)
- net EN: no longer Q1.3 (C)
- net GND: now also J1.3 (P3), C12.2, C14.2, C15.2, C18.2, C19.2, C20.2, C21.2, C22.2; no longer J1.4 (P4)
- net GPIO0: now also J2.2 (P2); no longer J1.1 (P1)
- net GPIO16: now also J1.1 (P1); no longer J2.1 (P1)
- net GPIO2: now also J2.1 (P1); no longer J1.2 (P2)
- net MISO: now also J4.6 (P6); no longer J4.5 (P5)
- net REST: now also Q1.3 (C)
- net SCLK: now also J4.5 (P5); no longer J4.6 (P6)
- net VBAT: now also C12.1, C14.1
- net at D4.1 (K), D5.1 (K), U7.3 (IN): now also C15.1, C18.1
Other:
- note added: "MISO"
- note added: "MOSI"
- note added: "SCK"
- note added: "SS"
- moved on the sheet: D4, D5, D8, J1, J4, R18, U7

Commit message: complete pcb source
Parts:
- removed C12, C14, C15, C18, C19, C20, C21, C22: C, esp8266:C_0603, symbol C
- removed D3: LED, LEDs:LED_0603, symbol LED_Small_ALT
- removed R16: 470, esp8266:R_0603, symbol R
- added C12, C14: 10uF, Capacitors_SMD:CP_Elec_4x5.3, symbol CP1
- added C15, C18: 22uF, Capacitors_SMD:CP_Elec_4x5.3, symbol CP1
- D7: footprint Diodes_SMD:D_SOD-123 -> Diodes_SMD:D_SOD-323
- SW1, SW2: footprint esp8266:Tact_Switch_TS6X3.6 -> esp8266:micro-buttom
Connections:
- net 3V3: now also C15.1
- net 5V: now also C18.1
- net GND: now also C12.2, C14.2, C15.2, C18.2
- net VBAT: now also C12.1
- net at D4.1 (K), D5.1 (K), U7.3 (IN): now also C14.1
- no-connect marks 22 -> 23
Changed lines of the file:
@@
 F 0 "SW1" H 6950 2150 50  0000 L CNN
 F 1 "SW_Push" H 6900 1990 50  0000 C CNN
-F 2 "esp8266:Tact_Switch_TS6X3.6" H 6900 2250 50  0001 C CNN
+F 2 "esp8266:micro-buttom" H 6900 2250 50  0001 C CNN
 F 3 "" H 6900 2250 50  0001 C CNN
 	1    6900 2050
@@
 F 0 "SW2" H 7550 2100 50  0000 L CNN
 F 1 "SW_Push" H 7500 1940 50  0000 C CNN
-F 2 "esp8266:Tact_Switch_TS6X3.6" H 7500 2200 50  0001 C CNN
+F 2 "esp8266:micro-buttom" H 7500 2200 50  0001 C CNN
 F 3 "" H 7500 2200 50  0001 C CNN
 	1    7500 2000
@@
 VBAT
 $Comp
-L mcp73831 U5
-U 1 1 59F0B81A
-P 9000 3700
-F 0 "U5" H 9100 4100 60  0000 C CNN
-F 1 "mcp73831" H 8900 3600 60  0000 C CNN
-F 2 "TO_SOT_Packages_SMD:SOT-23-5" H 9000 3700 60  0001 C CNN
-F 3 "" H 9000 3700 60  0001 C CNN
-	1    9000 3700
-	1    0    0    -1
-$EndComp
-$Comp
 L R R17
 U 1 1 59F0BAE6
@@
 F 0 "D7" H 10450 3380 50  0000 L CNN
 F 1 "BAT60JFILM" V 10500 2800 50  0000 L CNN
-F 2 "Diodes_SMD:D_SOD-123" V 10500 3300 50  0001 C CNN
+F 2 "Diodes_SMD:D_SOD-323" V 10500 3300 50  0001 C CNN
 F 3 "" V 10500 3300 50  0001 C CNN
 	1    10500 3300
@@
 Text GLabel 10600 3450 2    60   Input ~ 0
 VBAT
-$Comp
-L LED_Small_ALT D3
-U 1 1 59F1B94D
-P 8150 3600
-F 0 "D3" V 8100 3725 50  0000 L CNN
-F 1 "LED" H 7975 3500 50  0000 L CNN
-F 2 "LEDs:LED_0603" V 8150 3600 50  0001 C CNN
-F 3 "" V 8150 3600 50  0001 C CNN
-	1    8150 3600
-	0    -1   -1   0
-$EndComp
-$Comp
-L R R16
-U 1 1 59F1BAA4
-P 8350 3800
-F 0 "R16" V 8430 3800 50  0000 C CNN
-F 1 "470" V 8350 3800 50  0000 C CNN
-F 2 "esp8266:R_0603" V 8280 3800 50  0001 C CNN
-F 3 "" H 8350 3800 50  0001 C CNN
-	1    8350 3800
-	0    1    1    0
-$EndComp
 $Comp
 L LED_Small D8
@@
 Text Notes 7550 5950 0    60   ~ 0
 ADC IN
-$Comp
-L C C18
-U 1 1 59F5AC27
-P 8850 1350
-F 0 "C18" H 8875 1450 50  0000 L CNN
-F 1 "C" H 8875 1250 50  0000 L CNN
-F 2 "esp8266:C_0603" H 8888 1200 50  0001 C CNN
-F 3 "" H 8850 1350 50  0001 C CNN
-	1    8850 1350
-	1    0    0    -1
-$EndComp
-$Comp
-L C C15
-U 1 1 59F5ACC4
-P 8650 1350
-F 0 "C15" H 8675 1450 50  0000 L CNN
-F 1 "C" H 8675 1250 50  0000 L CNN
-F 2 "esp8266:C_0603" H 8688 1200 50  0001 C CNN
-F 3 "" H 8650 1350 50  0001 C CNN
-	1    8650 1350
-	1    0    0    -1
-$EndComp
-$Comp
-L C C21
-U 1 1 59F5B90C
-P 10400 1350
-F 0 "C21" H 10425 1450 50  0000 L CNN
-F 1 "C" H 10425 1250 50  0000 L CNN
-F 2 "esp8266:C_0603" H 10438 1200 50  0001 C CNN
-F 3 "" H 10400 1350 50  0001 C CNN
-	1    10400 1350
-	1    0    0    -1
-$EndComp
-$Comp
-L C C22
-U 1 1 59F5B9AB
-P 10600 1350
-F 0 "C22" H 10625 1450 50  0000 L CNN
-F 1 "C" H 10625 1250 50  0000 L CNN
-F 2 "esp8266:C_0603" H 10638 1200 50  0001 C CNN
-F 3 "" H 10600 1350 50  0001 C CNN
-	1    10600 1350
-	1    0    0    -1
-$EndComp
-$Comp
-L C C14
-U 1 1 59F5C166
-P 8500 2450
-F 0 "C14" H 8525 2550 50  0000 L CNN
-F 1 "C" H 8525 2350 50  0000 L CNN
-F 2 "esp8266:C_0603" H 8538 2300 50  0001 C CNN
-F 3 "" H 8500 2450 50  0001 C CNN
-	1    8500 2450
-	1    0    0    -1
-$EndComp
-$Comp
-L C C12
-U 1 1 59F5C207
-P 8300 2450
-F 0 "C12" H 8325 2550 50  0000 L CNN
-F 1 "C" H 8325 2350 50  0000 L CNN
-F 2 "esp8266:C_0603" H 8338 2300 50  0001 C CNN
-F 3 "" H 8300 2450 50  0001 C CNN
-	1    8300 2450
-	1    0    0    -1
-$EndComp
-$Comp
-L C C20
-U 1 1 59F5CDA6
-P 10250 2450
-F 0 "C20" H 10275 2550 50  0000 L CNN
-F 1 "C" H 10275 2350 50  0000 L CNN
-F 2 "esp8266:C_0603" H 10288 2300 50  0001 C CNN
-F 3 "" H 10250 2450 50  0001 C CNN
-	1    10250 2450
-	1    0    0    -1
-$EndComp
-$Comp
-L C C19
-U 1 1 59F5D11F
-P 10000 2450
-F 0 "C19" H 10025 2550 50  0000 L CNN
-F 1 "C" H 10025 2350 50  0000 L CNN
-F 2 "esp8266:C_0603" H 10038 2300 50  0001 C CNN
-F 3 "" H 10000 2450 50  0001 C CNN
-	1    10000 2450
-	1    0    0    -1
-$EndComp
 Wire Wire Line
 	7500 1650 7500 1800
@@
 Wire Wire Line
 	9650 1550 9650 1650
-Wire Wire Line
-	8650 1600 10600 1600
-Wire Wire Line
-	8850 1600 8850 1500
 Connection ~ 9650 1600
-Wire Wire Line
-	10400 1600 10400 1500
-Wire Wire Line
-	10400 1200 10400 1150
-Connection ~ 10400 1150
-Connection ~ 8850 1150
 Wire Wire Line
 	3800 3000 3650 3000
@@
 Wire Wire Line
 	9250 2650 9250 2750
-Wire Wire Line
-	8300 2700 10250 2700
-Wire Wire Line
-	8500 2700 8500 2600
 Connection ~ 9250 2700
 Wire Wire Line
-	10000 2700 10000 2600
-Wire Wire Line
-	10000 2300 10000 2250
-Wire Wire Line
 	9950 2250 10700 2250
-Connection ~ 10000 2250
 Wire Wire Line
 	10700 2250 10700 2100
-Connection ~ 10250 2250
 Wire Wire Line
 	8100 2250 8550 2250
@@
 Connection ~ 9700 3450
 Wire Wire Line
-	8500 2250 8500 2300
+	8500 2250 8500 2350
 Connection ~ 8500 2250
-Wire Wire Line
-	8850 1150 8850 1200
 Connection ~ 7900 3450
 Wire Wire Line
@@
 Wire Wire Line
 	10400 3450 10600 3450
-Wire Wire Line
-	8150 3200 8150 3500
 Wire Wire Line
 	8150 3200 11050 3200
@@
 	11050 3950 11050 3850
 Connection ~ 10500 3950
-Wire Wire Line
-	8150 3700 8150 3800
-Wire Wire Line
-	8150 3800 8200 3800
-Wire Wire Line
-	8500 3650 8500 3800
 Wire Bus Line
 	5600 2550 5600 4250
@@
 Wire Wire Line
 	10650 4900 10600 4900
-Wire Wire Line
-	8650 1200 8650 1150
-Connection ~ 8650 1150
-Wire Wire Line
-	8650 1500 8650 1600
-Connection ~ 8850 1600
-Wire Wire Line
-	10600 1200 10600 1150
-Connection ~ 10600 1150
-Wire Wire Line
-	10600 1600 10600 1500
-Connection ~ 10400 1600
 Connection ~ 10500 2250
 Wire Wire Line
-	10250 2300 10250 2250
-Wire Wire Line
-	10250 2700 10250 2600
-Connection ~ 10000 2700
-Wire Wire Line
-	8300 2300 8300 2250
-Connection ~ 8300 2250
-Wire Wire Line
-	8300 2600 8300 2700
+	9900 5900 9450 5900
+Wire Wire Line
+	9800 5100 9800 5150
+$Comp
+L CP1 C12
+U 1 1 59F9F26A
+P 8500 2500
+F 0 "C12" H 8525 2600 50  0000 L CNN
+F 1 "10uF" H 8525 2400 50  0000 L CNN
+F 2 "Capacitors_SMD:CP_Elec_4x5.3" H 8500 2500 50  0001 C CNN
+F 3 "" H 8500 2500 50  0001 C CNN
+	1    8500 2500
+	1    0    0    -1
+$EndComp
+Wire Wire Line
+	8500 2650 8500 2700
 Connection ~ 8500 2700
 Wire Wire Line
-	9900 5900 9450 5900
-Wire Wire Line
-	9800 5100 9800 5150
+	8500 2700 10050 2700
+$Comp
+L CP1 C15
+U 1 1 59F9FDF4
+P 10050 2500
+F 0 "C15" H 10075 2600 50  0000 L CNN
+F 1 "22uF" H 10075 2400 50  0000 L CNN
+F 2 "Capacitors_SMD:CP_Elec_4x5.3" H 10050 2500 50  0001 C CNN
+F 3 "" H 10050 2500 50  0001 C CNN
+	1    10050 2500
+	1    0    0    -1
+$EndComp
+Wire Wire Line
+	10050 2350 10050 2250
+Connection ~ 10050 2250
+Wire Wire Line
+	10050 2700 10050 2650
+$Comp
+L CP1 C18
+U 1 1 59FA0E70
+P 10550 1400
+F 0 "C18" H 10575 1500 50  0000 L CNN
+F 1 "22uF" H 10575 1300 50  0000 L CNN
+F 2 "Capacitors_SMD:CP_Elec_4x5.3" H 10550 1400 50  0001 C CNN
+F 3 "" H 10550 1400 50  0001 C CNN
+	1    10550 1400
+	1    0    0    -1
+$EndComp
+$Comp
+L CP1 C14
+U 1 1 59FA0F68
+P 8800 1400
+F 0 "C14" H 8825 1500 50  0000 L CNN
+F 1 "10uF" H 8825 1300 50  0000 L CNN
+F 2 "Capacitors_SMD:CP_Elec_4x5.3" H 8800 1400 50  0001 C CNN
+F 3 "" H 8800 1400 50  0001 C CNN
+	1    8800 1400
+	1    0    0    -1
+$EndComp
+Wire Wire Line
+	8800 1250 8800 1150
+Connection ~ 8800 1150
+Wire Wire Line
+	8800 1550 8800 1600
+Wire Wire Line
+	8800 1600 10550 1600
+Wire Wire Line
+	10550 1600 10550 1550
+Wire Wire Line
+	10550 1250 10550 1150
+Connection ~ 10550 1150
+Wire Wire Line
+	8150 3450 8150 3200
+$Comp
+L mcp73831 U5
+U 1 1 59F0B81A
+P 9000 3700
+F 0 "U5" H 9100 4100 60  0000 C CNN
+F 1 "mcp73831" H 8900 3600 60  0000 C CNN
+F 2 "TO_SOT_Packages_SMD:SOT-23-5" H 9000 3700 60  0001 C CNN
+F 3 "" H 9000 3700 60  0001 C CNN
+	1    9000 3700
+	1    0    0    -1
+$EndComp
+NoConn ~ 8500 3650
 $EndSCHEMATC

Commit message: xap xep linh kien
Parts:
- removed BT1: Battery, Pin_Headers:Pin_Header_Straight_2x01_Pitch2.00mm, symbol Battery_Cell
- removed C14: 10uF, Capacitors_SMD:CP_Elec_4x5.3, symbol CP1
- removed C16: 4.7uF, esp8266:C_0603, symbol C
- removed C17: 1uF, esp8266:C_0603, symbol C
- removed C18: 22uF, Capacitors_SMD:CP_Elec_4x5.3, symbol CP1
- removed D2: ZENER_3V3, Diodes_SMD:D_SOD-323_HandSoldering, symbol D_Schottky_ALT
- removed D4: SS34, esp8266:do214aa-g, symbol D_Schottky_Small
- removed D7: BAT60JFILM, Diodes_SMD:D_SOD-323, symbol D_Schottky_Small
- removed J1, J6: CONN_01X04, Pin_Headers:Pin_Header_Straight_1x04_Pitch2.54mm, symbol CONN_01X04
- removed J2: CONN_01X02, Pin_Headers:Pin_Header_Straight_1x02_Pitch2.54mm, symbol CONN_01X02
- removed J3, J5: CONN_01X08, Pin_Headers:Pin_Header_Straight_1x08_Pitch2.54mm, symbol CONN_01X08
- removed J4: CONN_01X06, Pin_Headers:Pin_Header_Straight_1x06_Pitch2.54mm, symbol CONN_01X06
- removed R17: 2K, esp8266:R_0603, symbol R
- removed R19: 100k, esp8266:R_0603, symbol R
- removed U5: mcp73831, TO_SOT_Packages_SMD:SOT-23-5, symbol mcp73831
- removed U7: AMS1117-3.3, TO_SOT_Packages_SMD:SOT-223, symbol AMS1117-3.3
- removed U8: MOSFET-P, esp8266:SOT-23_standar, symbol MOSFET-P
- added J1, J2: CONN_01X10, Pin_Headers:Pin_Header_Straight_1x10_Pitch2.54mm, symbol CONN_01X10
- C12: value 10uF -> 10uF TANT; footprint Capacitors_SMD:CP_Elec_4x5.3 -> Capacitors_SMD:C_1206
- C13: value 4.7uF -> 100nF
- C15: value 22uF -> 10uF TANT; footprint Capacitors_SMD:CP_Elec_4x5.3 -> Capacitors_SMD:C_1206
- D5: value SS34 -> 1n5819; footprint esp8266:do214aa-g -> Diodes_SMD:D_SOD-123
- SW1, SW2: footprint esp8266:micro-buttom -> esp8266:tactile switches
- U3: footprint Housings_DFN_QFN:QFN-28-1EP_5x5mm_Pitch0.5mm -> esp8266:cp2102
- U4: footprint Housings_SOIC:SOIJ-8_5.3x5.3mm_Pitch1.27mm -> Housings_SOIC:SOIC-8_3.9x4.9mm_Pitch1.27mm
Connections:
- net 5V is gone; now on net 3V3: C13.1
- net VBAT is gone; now on net VCC: C12.1, U6.3 (IN)
- net 3V3: now also U4.8 (VCC), J1.10 (P10), J2.4 (P4)
- net ADC_EX: now also J2.2 (P2)
- net EN: now also J2.5 (P5)
- net GND: now also U3.29 (GND), U4.4 (GND), J1.9 (P9), J2.10 (P10), J2.3 (P3)
- net GPIO0: now also J2.7 (P7)
- net GPIO12: now also J1.2 (P2)
- net GPIO13: now also J1.3 (P3)
- net GPIO14: now also J1.1 (P1)
- net GPIO15: now also J1.4 (P4)
- net GPIO16: now also J2.1 (P1)
- net GPIO2: now also J2.8 (P8)
- net GPIO4: now also J1.7 (P7)
- net GPIO5: now also J1.8 (P8)
- net REST: now also J2.6 (P6)
- net RXD: now also J1.5 (P5)
- net TXD: now also J1.6 (P6)
- net VUSB: now also J2.9 (P9); no longer C6.1, C8.1, U3.8 (VBUS)
- net VCC: now reaches D5.1 (K)
- net VCC: now also C6.1, C8.1, U3.8 (VBUS)
- no-connect marks 23 -> 21
Other:
- note removed: "SPI FLASH"
- moved on the sheet: C12, C15, D5, D8, R18, U6

Commit message: complete pcb ver2.0
Parts:
- SW1, SW2: footprint esp8266:tactile switches -> esp8266:nut_nhan_ngang
Connections:
- net ADC_EX: now also J2.9 (P9); no longer J2.2 (P2)
- net EN: now also J2.8 (P8); no longer J2.5 (P5)
- net GND: now also J2.1 (P1), J2.2 (P2); no longer J2.10 (P10), J2.3 (P3)
- net GPIO0: now also J2.5 (P5); no longer J2.7 (P7)
- net GPIO16: now also J2.7 (P7); no longer J2.1 (P1)
- net GPIO2: now also J2.6 (P6); no longer J2.8 (P8)
- net REST: now also J2.10 (P10); no longer J2.6 (P6)
- net VCC: now also J2.3 (P3)
- net VUSB: no longer J2.9 (P9)
Other:
- note removed: "MISO"
- note removed: "MOSI"
- note removed: "OLED"
- note removed: "SCK"
- note removed: "SS"
Changed lines of the file:
@@
 F 0 "SW1" H 6950 2150 50  0000 L CNN
 F 1 "SW_Push" H 6900 1990 50  0000 C CNN
-F 2 "esp8266:tactile switches" H 6900 2250 50  0001 C CNN
+F 2 "esp8266:nut_nhan_ngang" H 6900 2250 50  0001 C CNN
 F 3 "" H 6900 2250 50  0001 C CNN
 	1    6900 2050
@@
 F 0 "SW2" H 7550 2100 50  0000 L CNN
 F 1 "SW_Push" H 7500 1940 50  0000 C CNN
-F 2 "esp8266:tactile switches" H 7500 2200 50  0001 C CNN
+F 2 "esp8266:nut_nhan_ngang" H 7500 2200 50  0001 C CNN
 F 3 "" H 7500 2200 50  0001 C CNN
 	1    7500 2000
@@
 Text GLabel 8350 5300 2    60   Input ~ 0
 RXD
+Text GLabel 9450 5800 2    60   Input ~ 0
+REST
+Text GLabel 9450 5600 2    60   Input ~ 0
+EN
+Text GLabel 9450 5700 2    60   Input ~ 0
+ADC_EX
+Text GLabel 9450 5500 2    60   Input ~ 0
+GPIO16
+Text GLabel 9450 5300 2    60   Input ~ 0
+GPIO0
 Text GLabel 9450 5400 2    60   Input ~ 0
-REST
-Text GLabel 9450 5300 2    60   Input ~ 0
-EN
-Text GLabel 9450 5000 2    60   Input ~ 0
-ADC_EX
-Text GLabel 9450 4900 2    60   Input ~ 0
-GPIO16
-Text GLabel 9450 5500 2    60   Input ~ 0
-GPIO0
-Text GLabel 9450 5600 2    60   Input ~ 0
 GPIO2
 Text GLabel 9450 5200 2    60   Input ~ 0
@@
 L GND #PWR015
 U 1 1 59F32D9B
-P 9800 5150
-F 0 "#PWR015" H 9800 4900 50  0001 C CNN
-F 1 "GND" H 9800 5000 50  0000 C CNN
-F 2 "" H 9800 5150 50  0001 C CNN
-F 3 "" H 9800 5150 50  0001 C CNN
-	1    9800 5150
+P 10050 5200
+F 0 "#PWR015" H 10050 4950 50  0001 C CNN
+F 1 "GND" H 10050 5050 50  0000 C CNN
+F 2 "" H 10050 5200 50  0001 C CNN
+F 3 "" H 10050 5200 50  0001 C CNN
+	1    10050 5200
 	-1   0    0    -1
 $EndComp
-Text Notes 10900 6000 2    79   ~ 16
-SOURCE
-Text Notes 9650 6350 2    79   ~ 16
-OLED
 $Comp
 L GND #PWR016
@@
 	1    0    0    -1
 $EndComp
-Text Notes 8800 5250 0    60   ~ 0
-SCK
-Text Notes 8800 5150 0    60   ~ 0
-MISO
-Text Notes 8800 4950 0    60   ~ 0
-MOSI
-Text Notes 8800 5050 0    60   ~ 0
-SS
-Text Notes 7550 5950 0    60   ~ 0
-ADC IN
 Wire Wire Line
 	7500 1650 7500 1800
@@
 	9450 5200 9350 5200
 Wire Wire Line
-	9350 5100 9800 5100
-Wire Wire Line
-	9450 5000 9350 5000
-Wire Wire Line
-	9450 4900 9350 4900
+	9350 4900 10050 4900
 Wire Wire Line
 	7500 2200 7500 2300
@@
 	900  2250 900  2200
 Connection ~ 10850 2450
-Wire Wire Line
-	9800 5100 9800 5150
 $Comp
 L CP1 C12
@@
 	1    0    0    -1
 $EndComp
-Text GLabel 9450 5700 2    60   Input ~ 0
-VUSB
-$Comp
-L GND #PWR020
-U 1 1 59FB00DA
-P 9800 5850
-F 0 "#PWR020" H 9800 5600 50  0001 C CNN
-F 1 "GND" H 9800 5700 50  0000 C CNN
-F 2 "" H 9800 5850 50  0001 C CNN
-F 3 "" H 9800 5850 50  0001 C CNN
-	1    9800 5850
-	1    0    0    -1
-$EndComp
+Text GLabel 9450 5100 2    60   Input ~ 0
+VCC
 Text GLabel 1450 4750 0    60   Input ~ 0
 VUSB
@@
 	9350 5700 9450 5700
 Wire Wire Line
-	9350 5800 9800 5800
-Wire Wire Line
-	9800 5800 9800 5850
-Wire Wire Line
 	3200 7300 3200 7450
 Wire Wire Line
 	3200 7450 3300 7450
 Connection ~ 3300 7450
+Wire Wire Line
+	10050 4900 10050 5200
+Wire Wire Line
+	9450 5800 9350 5800
+Wire Wire Line
+	9450 5100 9350 5100
+Wire Wire Line
+	9350 5000 10050 5000
+Connection ~ 10050 5000
 $EndSCHEMATC
